File: kicad/i2c_level_shift.kicad_sch (KiCad schematic)
At the start: 4 parts, among them Q3101 NMOS

Commit message: Added Digikey references
Parts:
- Q3101: Digikey (none) -> SQ1922AEEH-T1_GE3CT-ND; Purpose (none) -> I2C level shift
Changed lines of the file:
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@@
+      (effects (font (size 1.27 1.27)) hide)
+    )
+    (property "Digikey" "SQ1922AEEH-T1_GE3CT-ND" (id 4) (at 144.78 124.46 0)
+      (effects (font (size 1.27 1.27)) hide)
+    )
+    (property "Purpose" "I2C level shift" (id 5) (at 144.78 124.46 0)
       (effects (font (size 1.27 1.27)) hide)
     )
@@
       (effects (font (size 1.27 1.27)) hide)
     )
+    (property "Digikey" "SQ1922AEEH-T1_GE3CT-ND" (id 4) (at 144.78 86.36 0)
+      (effects (font (size 1.27 1.27)) hide)
+    )
+    (property "Purpose" "I2C level shift" (id 5) (at 144.78 86.36 0)
+      (effects (font (size 1.27 1.27)) hide)
+    )

Commit message: Updated Digikey part numbers
Darn supply chain crisis :(
Parts:
- Q3101: Digikey SQ1922AEEH-T1_GE3CT-ND -> UM6K1NTNCT-ND
- R3101, R3102: Digikey (none) -> P5.1KJCT-ND; Purpose (none) -> I2C level shifted pullup
Changed lines of the file:
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@@
       (effects (font (size 1.27 1.27)) hide)
     )
-    (property "Digikey" "SQ1922AEEH-T1_GE3CT-ND" (id 4) (at 144.78 124.46 0)
+    (property "Digikey" "UM6K1NTNCT-ND" (id 4) (at 144.78 124.46 0)
       (effects (font (size 1.27 1.27)) hide)
     )
@@
       (effects (font (size 1.524 1.524)) hide)
     )
+    (property "Purpose" "I2C level shifted pullup" (id 4) (at 127 82.55 0)
+      (effects (font (size 1.27 1.27)) hide)
+    )
+    (property "Digikey" "P5.1KJCT-ND" (id 5) (at 127 82.55 0)
+      (effects (font (size 1.27 1.27)) hide)
+    )
     (pin "1")
     (pin "2")
@@
       (effects (font (size 1.524 1.524)) hide)
     )
+    (property "Purpose" "I2C level shifted pullup" (id 4) (at 127 120.65 0)
+      (effects (font (size 1.27 1.27)) hide)
+    )
+    (property "Digikey" "P5.1KJCT-ND" (id 5) (at 127 120.65 0)
+      (effects (font (size 1.27 1.27)) hide)
+    )
     (pin "1")
     (pin "2")
@@
       (effects (font (size 1.27 1.27)) hide)
     )
-    (property "Digikey" "SQ1922AEEH-T1_GE3CT-ND" (id 4) (at 144.78 86.36 0)
+    (property "Digikey" "UM6K1NTNCT-ND" (id 4) (at 144.78 86.36 0)
       (effects (font (size 1.27 1.27)) hide)
     )
@@
       (effects (font (size 1.27 1.27)) hide)
     )
-    (pin "1")
-    (pin "2")
-    (pin "6")
+    (pin "3")
+    (pin "4")
+    (pin "5")
   )
 )
