File: kicad/ICM-42688.kicad_sch (KiCad schematic)
At the start: 4 parts, among them U2701 ICM-42688

Commit message: Broke down sensor block into a tree of sheets
Parts:
- renumbered C2705 to C3205, C2706 to C3206, C2708 to C3208, U2701 to U3201
Changed lines of the file:
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@@
   (symbol (lib_id "KwanSystems:ICM-42688") (at 114.3 62.23 0)
     (in_bom yes) (on_board yes) (fields_autoplaced)
-    (property "Reference" "U2701" (id 0) (at 129.4537 54.9867 0))
+    (property "Reference" "U3201" (id 0) (at 129.4537 54.9867 0))
     (property "Value" "ICM-42688" (id 1) (at 129.4537 57.7618 0))
     (property "Footprint" "KwanSystems:QFN50P300X250X97-14N" (id 2) (at 147.32 67.31 0)
@@
   (symbol (lib_id "Device:C") (at 154.94 82.55 0)
     (in_bom yes) (on_board yes) (fields_autoplaced)
-    (property "Reference" "C2706" (id 0) (at 157.861 81.6415 0)
+    (property "Reference" "C3206" (id 0) (at 157.861 81.6415 0)
       (effects (font (size 1.27 1.27)) (justify left))
     )
@@
   (symbol (lib_id "Device:C") (at 116.84 82.55 0)
     (in_bom yes) (on_board yes) (fields_autoplaced)
-    (property "Reference" "C2705" (id 0) (at 119.761 81.6415 0)
+    (property "Reference" "C3205" (id 0) (at 119.761 81.6415 0)
       (effects (font (size 1.27 1.27)) (justify left))
     )
@@
   (symbol (lib_id "Device:C") (at 142.24 82.55 0)
     (in_bom yes) (on_board yes) (fields_autoplaced)
-    (property "Reference" "C2708" (id 0) (at 145.161 81.6415 0)
+    (property "Reference" "C3208" (id 0) (at 145.161 81.6415 0)
       (effects (font (size 1.27 1.27)) (justify left))
     )

Commit message: One shining moment
Commit board while it still works
Parts:
- C1205: renamed from C3205; Digikey 399-C0603C103J5RAC7867CT-ND -> 399-C0402C103J5RAC7867CT-ND
- C1206: renamed from C3206; Digikey 399-13137-1-ND -> 399-11617-1-ND
- C1208: renamed from C3208; Digikey 399-C0603C104M5RAC7867CT-ND -> 399-C0402C104K4RAC7411CT-ND
- U1201: renamed from U3201; Digikey (none) -> 1428-ICM-42688-PCT-ND; Purpose (none) -> Inertial Sensor 6DoF
Changed lines of the file:
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@@
   (symbol (lib_id "KwanSystems:ICM-42688") (at 114.3 62.23 0)
     (in_bom yes) (on_board yes) (fields_autoplaced)
-    (property "Reference" "U3201" (id 0) (at 129.4537 54.9867 0))
+    (property "Reference" "U1201" (id 0) (at 129.4537 54.9867 0))
     (property "Value" "ICM-42688" (id 1) (at 129.4537 57.7618 0))
     (property "Footprint" "KwanSystems:QFN50P300X250X97-14N" (id 2) (at 147.32 67.31 0)
@@
     )
     (property "Datasheet" "https://invensense.tdk.com/download-pdf/icm-42688-p-datasheet/" (id 3) (at 151.13 72.39 0)
+      (effects (font (size 1.27 1.27)) hide)
+    )
+    (property "Digikey" "1428-ICM-42688-PCT-ND" (id 4) (at 114.3 62.23 0)
+      (effects (font (size 1.27 1.27)) hide)
+    )
+    (property "Purpose" "Inertial Sensor 6DoF" (id 5) (at 114.3 62.23 0)
       (effects (font (size 1.27 1.27)) hide)
     )
@@
   (symbol (lib_id "Device:C") (at 154.94 82.55 0)
     (in_bom yes) (on_board yes) (fields_autoplaced)
-    (property "Reference" "C3206" (id 0) (at 157.861 81.6415 0)
+    (property "Reference" "C1206" (id 0) (at 157.861 81.6415 0)
       (effects (font (size 1.27 1.27)) (justify left))
     )
@@
       (effects (font (size 1.27 1.27)) hide)
     )
-    (property "Digikey" "399-13137-1-ND" (id 4) (at 154.94 82.55 0)
+    (property "Digikey" "399-11617-1-ND" (id 4) (at 154.94 82.55 0)
       (effects (font (size 1.27 1.27)) hide)
     )
@@
   (symbol (lib_id "Device:C") (at 116.84 82.55 0)
     (in_bom yes) (on_board yes) (fields_autoplaced)
-    (property "Reference" "C3205" (id 0) (at 119.761 81.6415 0)
+    (property "Reference" "C1205" (id 0) (at 119.761 81.6415 0)
       (effects (font (size 1.27 1.27)) (justify left))
     )
@@
       (effects (font (size 1.27 1.27)) hide)
     )
-    (property "Digikey" "399-C0603C103J5RAC7867CT-ND" (id 4) (at 116.84 82.55 0)
+    (property "Digikey" "399-C0402C103J5RAC7867CT-ND" (id 4) (at 116.84 82.55 0)
       (effects (font (size 1.27 1.27)) hide)
     )
@@
   (symbol (lib_id "Device:C") (at 142.24 82.55 0)
     (in_bom yes) (on_board yes) (fields_autoplaced)
-    (property "Reference" "C3208" (id 0) (at 145.161 81.6415 0)
+    (property "Reference" "C1208" (id 0) (at 145.161 81.6415 0)
       (effects (font (size 1.27 1.27)) (justify left))
     )
@@
       (effects (font (size 1.27 1.27)) hide)
     )
-    (property "Digikey" "399-C0603C104M5RAC7867CT-ND" (id 4) (at 142.24 82.55 0)
+    (property "Digikey" "399-C0402C104K4RAC7411CT-ND" (id 4) (at 142.24 82.55 0)
       (effects (font (size 1.27 1.27)) hide)
     )

Commit message: Updated symbol
This incorporates the change in the library, to offset the NC pins and satisfy the ERC
Parts:
- renumbered C1205 to C3205, C1206 to C3206, C1208 to C3208, U1201 to U3201
Connections:
- now unconnected: U3201.10 (RESV), U3201.11 (RESV), U3201.2 (RESV), U3201.3 (RESV), U3201.7 (RESV)
Changed lines of the file:
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@@
   (symbol (lib_id "KwanSystems:ICM-42688") (at 114.3 62.23 0)
     (in_bom yes) (on_board yes) (fields_autoplaced)
-    (property "Reference" "U1201" (id 0) (at 129.4537 54.9867 0))
+    (property "Reference" "U3201" (id 0) (at 129.4537 54.9867 0))
     (property "Value" "ICM-42688" (id 1) (at 129.4537 57.7618 0))
     (property "Footprint" "KwanSystems:QFN50P300X250X97-14N" (id 2) (at 147.32 67.31 0)
@@
   (symbol (lib_id "Device:C") (at 154.94 82.55 0)
     (in_bom yes) (on_board yes) (fields_autoplaced)
-    (property "Reference" "C1206" (id 0) (at 157.861 81.6415 0)
+    (property "Reference" "C3206" (id 0) (at 157.861 81.6415 0)
       (effects (font (size 1.27 1.27)) (justify left))
     )
@@
   (symbol (lib_id "Device:C") (at 116.84 82.55 0)
     (in_bom yes) (on_board yes) (fields_autoplaced)
-    (property "Reference" "C1205" (id 0) (at 119.761 81.6415 0)
+    (property "Reference" "C3205" (id 0) (at 119.761 81.6415 0)
       (effects (font (size 1.27 1.27)) (justify left))
     )
@@
   (symbol (lib_id "Device:C") (at 142.24 82.55 0)
     (in_bom yes) (on_board yes) (fields_autoplaced)
-    (property "Reference" "C1208" (id 0) (at 145.161 81.6415 0)
+    (property "Reference" "C3208" (id 0) (at 145.161 81.6415 0)
       (effects (font (size 1.27 1.27)) (justify left))
     )
