File: kicad/sensors.kicad_sch (KiCad schematic)
At the start: 0 parts

Commit message: Checkin before branch
Connections:
- no-connect marks 6 -> 5
Other:
- added sheet Int Level Shift1 (i2c_level_shift.kicad_sch)
- added sheet Int Level Shift2 (i2c_level_shift.kicad_sch)
