File: kicad/GPS_rover.kicad_sch (KiCad schematic)
At the start: 15 parts, among them J201 SMA, J202 NormallyClosed, U201 ZED_F9R, Y401 ANN-MB-00

Commit message: Commit as-ordered shipometer 23.03
Parts:
- B201, C201, L201, R238, R239, U201: Number on hand (none) -> 1
- C236, C238: Mouser (none) -> 187-CL05A105KP5NNWC; Number on hand (none) -> 14+10
- D201, R253, Y401: Number on hand (none) -> 2
- J201: Number in cart (none) -> 1; Number on hand (none) -> 0
- J202: footprint KwanSystems:SolderJumper-2_P1.3mm_MaskBridged_RoundedPad1.0x1.5mm -> Jumper:SolderJumper-2_P1.3mm_Bridged_RoundedPad1.0x1.5mm
- R436: Number on hand (none) -> 12
Changed lines of the file:
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@@
+      (effects (font (size 1.27 1.27)) hide)
+    )
+    (property "Mouser" "187-CL05A105KP5NNWC" (id 6) (at 120.65 170.18 0)
+      (effects (font (size 1.27 1.27)) hide)
+    )
+    (property "Number on hand" "14+10" (id 7) (at 120.65 170.18 0)
       (effects (font (size 1.27 1.27)) hide)
     )
@@
     )
     (property "Purpose" "GPS input protection" (id 5) (at 167.64 66.04 0)
+      (effects (font (size 1.27 1.27)) hide)
+    )
+    (property "Number on hand" "1" (id 6) (at 167.64 66.04 0)
       (effects (font (size 1.27 1.27)) hide)
     )
@@
       (effects (font (size 1.27 1.27)) hide)
     )
+    (property "Number on hand" "1" (id 6) (at 156.21 154.94 0)
+      (effects (font (size 1.27 1.27)) hide)
+    )
     (pin "1")
     (pin "2")
@@
     )
     (property "Purpose" "GPS input protection" (id 5) (at 99.06 76.2 0)
+      (effects (font (size 1.27 1.27)) hide)
+    )
+    (property "Number on hand" "1" (id 6) (at 99.06 76.2 0)
       (effects (font (size 1.27 1.27)) hide)
     )
@@
       (effects (font (size 1.27 1.27)) hide)
     )
+    (property "Number on hand" "0" (id 6) (at 144.78 149.86 0)
+      (effects (font (size 1.27 1.27)) hide)
+    )
+    (property "Number in cart" "1" (id 7) (at 144.78 149.86 0)
+      (effects (font (size 1.27 1.27)) hide)
+    )
     (pin "1")
     (pin "2")
@@
       (effects (font (size 1.27 1.27)) hide)
     )
+    (property "Number on hand" "12" (id 8) (at 107.95 158.75 0)
+      (effects (font (size 1.27 1.27)) hide)
+    )
     (pin "1")
     (pin "2")
@@
     )
     (property "Purpose" "GPS input protection" (id 5) (at 99.06 78.74 0)
+      (effects (font (size 1.27 1.27)) hide)
+    )
+    (property "Number on hand" "1" (id 6) (at 99.06 78.74 0)
       (effects (font (size 1.27 1.27)) hide)
     )
@@
       (effects (font (size 1.27 1.27)) hide)
     )
+    (property "Number on hand" "1" (id 6) (at 156.21 167.64 0)
+      (effects (font (size 1.27 1.27)) hide)
+    )
     (pin "1")
     (pin "2")
@@
     )
     (property "Digikey" "672-ZED-F9R-02BCT-ND" (id 5) (at 129.54 63.5 0)
+      (effects (font (size 1.27 1.27)) hide)
+    )
+    (property "Number on hand" "1" (id 6) (at 129.54 63.5 0)
       (effects (font (size 1.27 1.27)) hide)
     )
@@
       (effects (font (size 1.27 1.27)) hide)
     )
+    (property "Number on hand" "2" (id 6) (at 163.83 138.43 0)
+      (effects (font (size 1.27 1.27)) hide)
+    )
     (pin "1")
   )
@@
     )
     (property "Digikey" "P27JCT-ND" (id 5) (at 168.91 162.56 0)
+      (effects (font (size 1.27 1.27)) hide)
+    )
+    (property "Number on hand" "" (id 6) (at 168.91 162.56 0)
       (effects (font (size 1.27 1.27)) hide)
     )
@@
       (effects (font (size 1.27 1.27)) hide)
     )
-    (property "Footprint" "KwanSystems:SolderJumper-2_P1.3mm_MaskBridged_RoundedPad1.0x1.5mm" (id 2) (at 160.02 162.56 0)
+    (property "Footprint" "Jumper:SolderJumper-2_P1.3mm_Bridged_RoundedPad1.0x1.5mm" (id 2) (at 160.02 162.56 0)
       (effects (font (size 1.27 1.27)) hide)
     )
@@
       (effects (font (size 1.27 1.27)) hide)
     )
+    (property "Mouser" "187-CL05A105KP5NNWC" (id 6) (at 73.66 81.28 0)
+      (effects (font (size 1.27 1.27)) hide)
+    )
+    (property "Number on hand" "14+10" (id 7) (at 73.66 81.28 0)
+      (effects (font (size 1.27 1.27)) hide)
+    )
     (pin "1")
     (pin "2")
@@
       (effects (font (size 1.27 1.27)) hide)
     )
+    (property "Number on hand" "2" (id 6) (at 167.64 88.9 0)
+      (effects (font (size 1.27 1.27)) hide)
+    )
     (pin "1")
     (pin "2")
@@
       (effects (font (size 1.27 1.27)) hide)
     )
+    (property "Number on hand" "1" (id 6) (at 107.95 172.72 0)
+      (effects (font (size 1.27 1.27)) hide)
+    )
     (pin "1")
     (pin "2")
@@
       (effects (font (size 1.27 1.27)) hide)
     )
+    (property "Number on hand" "2" (id 7) (at 107.95 144.78 0)
+      (effects (font (size 1.27 1.27)) hide)
+    )
     (pin "1")
     (pin "2")
@@
     )
     (property "Purpose" "GPS input protection" (id 5) (at 167.64 68.58 0)
+      (effects (font (size 1.27 1.27)) hide)
+    )
+    (property "Number on hand" "1" (id 6) (at 167.64 68.58 0)
       (effects (font (size 1.27 1.27)) hide)
     )
@@
       (effects (font (size 1.27 1.27)) hide)
     )
+    (property "Number on hand" "1" (id 6) (at 78.74 86.36 0)
+      (effects (font (size 1.27 1.27)) hide)
+    )
