File: kicad/regulator.kicad_sch (KiCad schematic)
At the start: 3 parts, among them U401 TCR2EF 3.3V

Commit message: Added BME280 and ICM20948 stamps
Parts:
- C401, C405: footprint Capacitor_SMD:C_0402_1005Metric -> Capacitor_SMD:C_0603_1608Metric
Changed lines of the file:
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@@
       (effects (font (size 1.27 1.27)) (justify left))
     )
-    (property "Footprint" "Capacitor_SMD:C_0402_1005Metric" (at 114.3 105.41 0)
+    (property "Footprint" "Capacitor_SMD:C_0603_1608Metric" (at 114.3 105.41 0)
       (effects (font (size 1.27 1.27)) hide)
     )
@@
       (effects (font (size 1.27 1.27)) (justify left))
     )
-    (property "Footprint" "Capacitor_SMD:C_0402_1005Metric" (at 144.78 109.22 0)
+    (property "Footprint" "Capacitor_SMD:C_0603_1608Metric" (at 144.78 109.22 0)
       (effects (font (size 1.27 1.27)) hide)
     )

Commit message: As ordered on 03 Apr 2023. Some but not all numbers-on-hand have been updated.
Parts:
- C401, C405: Digikey 399-C0402C105K9PAC7800CT-ND -> 399-C0603C105K4PAC7411CT-ND; Mouser 187-CL05A105KP5NNWC -> 80-C0603C105K4PAC; Number on hand 14+10 -> (none)
- U401: Number on hand 1 -> (none)
Changed lines of the file:
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@@
       (effects (font (size 1.27 1.27)) hide)
     )
-    (property "Number on hand" "1" (at 129.54 96.52 0)
+    (property "Number on hand" "" (at 129.54 96.52 0)
       (effects (font (size 1.27 1.27)) hide)
     )
@@
       (effects (font (size 1.27 1.27)) hide)
     )
-    (property "Datasheet" "~" (at 114.3 105.41 0)
+    (property "Datasheet" "https://connect.kemet.com:7667/gateway/IntelliData-ComponentDocumentation/1.0/download/datasheet/C0603C105K4PACTU" (at 114.3 105.41 0)
       (effects (font (size 1.27 1.27)) hide)
     )
-    (property "Digikey" "399-C0402C105K9PAC7800CT-ND" (at 114.3 105.41 0)
+    (property "Digikey" "399-C0603C105K4PAC7411CT-ND" (at 114.3 105.41 0)
       (effects (font (size 1.27 1.27)) hide)
     )
@@
       (effects (font (size 1.27 1.27)) hide)
     )
-    (property "Mouser" "187-CL05A105KP5NNWC" (at 114.3 105.41 0)
+    (property "Mouser" "80-C0603C105K4PAC" (at 114.3 105.41 0)
       (effects (font (size 1.27 1.27)) hide)
     )
-    (property "Number on hand" "14+10" (at 114.3 105.41 0)
+    (property "Number on hand" "" (at 114.3 105.41 0)
       (effects (font (size 1.27 1.27)) hide)
     )
@@
       (effects (font (size 1.27 1.27)) hide)
     )
-    (property "Datasheet" "~" (at 144.78 109.22 0)
+    (property "Datasheet" "https://connect.kemet.com:7667/gateway/IntelliData-ComponentDocumentation/1.0/download/datasheet/C0603C105K4PACTU" (at 144.78 109.22 0)
       (effects (font (size 1.27 1.27)) hide)
     )
-    (property "Digikey" "399-C0402C105K9PAC7800CT-ND" (at 144.78 109.22 0)
+    (property "Digikey" "399-C0603C105K4PAC7411CT-ND" (at 144.78 109.22 0)
       (effects (font (size 1.27 1.27)) hide)
     )
@@
       (effects (font (size 1.27 1.27)) hide)
     )
-    (property "Mouser" "187-CL05A105KP5NNWC" (at 144.78 109.22 0)
+    (property "Mouser" "80-C0603C105K4PAC" (at 144.78 109.22 0)
       (effects (font (size 1.27 1.27)) hide)
     )
-    (property "Number on hand" "14+10" (at 144.78 109.22 0)
+    (property "Number on hand" "" (at 144.78 109.22 0)
       (effects (font (size 1.27 1.27)) hide)
     )

Commit message: Updated numbers on hand and numbers in cart
Parts:
- C401, C405: Number in cart (none) -> 24; Number on hand (none) -> 0
- U401: Mouser (none) -> 998-MIC5317-3.3YD5TR; Number in cart (none) -> 5; Number on hand (none) -> 0
Changed lines of the file:
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@@
       (effects (font (size 1.27 1.27)) hide)
     )
-    (property "Number on hand" "" (at 129.54 96.52 0)
+    (property "Number on hand" "0" (at 129.54 96.52 0)
+      (effects (font (size 1.27 1.27)) hide)
+    )
+    (property "Mouser" "998-MIC5317-3.3YD5TR" (at 129.54 96.52 0)
+      (effects (font (size 1.27 1.27)) hide)
+    )
+    (property "Number in cart" "5" (at 129.54 96.52 0)
       (effects (font (size 1.27 1.27)) hide)
     )
@@
       (effects (font (size 1.27 1.27)) hide)
     )
-    (property "Number on hand" "" (at 114.3 105.41 0)
+    (property "Number on hand" "0" (at 114.3 105.41 0)
+      (effects (font (size 1.27 1.27)) hide)
+    )
+    (property "Number in cart" "24" (at 114.3 105.41 0)
       (effects (font (size 1.27 1.27)) hide)
     )
@@
       (effects (font (size 1.27 1.27)) hide)
     )
-    (property "Number on hand" "" (at 144.78 109.22 0)
+    (property "Number on hand" "0" (at 144.78 109.22 0)
       (effects (font (size 1.27 1.27)) hide)
     )
+    (property "Number in cart" "24" (at 144.78 109.22 0)
+      (effects (font (size 1.27 1.27)) hide)
+    )

Commit message: Updated number on hand, and added more Digikey/Mouser/Mfg numbers
Parts:
- C401, C405: Number in cart 24 -> (none); Number on hand 0 -> 24; Part Number (none) -> C0603C105K4PAC
- U401: Number in cart 5 -> (none); Number on hand 0 -> 5; Part Number (none) -> MIC5317-3.3YD5-TR
Changed lines of the file:
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@@
       (effects (font (size 1.27 1.27)) hide)
     )
-    (property "Number on hand" "0" (at 129.54 96.52 0)
+    (property "Number on hand" "5" (at 129.54 96.52 0)
       (effects (font (size 1.27 1.27)) hide)
     )
@@
       (effects (font (size 1.27 1.27)) hide)
     )
-    (property "Number in cart" "5" (at 129.54 96.52 0)
+    (property "Number in cart" "" (at 129.54 96.52 0)
+      (effects (font (size 1.27 1.27)) hide)
+    )
+    (property "Part Number" "MIC5317-3.3YD5-TR" (at 129.54 96.52 0)
       (effects (font (size 1.27 1.27)) hide)
     )
@@
       (effects (font (size 1.27 1.27)) hide)
     )
-    (property "Number on hand" "0" (at 114.3 105.41 0)
+    (property "Number on hand" "24" (at 114.3 105.41 0)
       (effects (font (size 1.27 1.27)) hide)
     )
-    (property "Number in cart" "24" (at 114.3 105.41 0)
+    (property "Number in cart" "" (at 114.3 105.41 0)
+      (effects (font (size 1.27 1.27)) hide)
+    )
+    (property "Part Number" "C0603C105K4PAC" (at 114.3 105.41 0)
       (effects (font (size 1.27 1.27)) hide)
     )
@@
       (effects (font (size 1.27 1.27)) hide)
     )
-    (property "Number on hand" "0" (at 144.78 109.22 0)
+    (property "Number on hand" "24" (at 144.78 109.22 0)
       (effects (font (size 1.27 1.27)) hide)
     )
-    (property "Number in cart" "24" (at 144.78 109.22 0)
+    (property "Number in cart" "" (at 144.78 109.22 0)
       (effects (font (size 1.27 1.27)) hide)
     )
+    (property "Part Number" "C0603C105K4PAC" (at 144.78 109.22 0)
+      (effects (font (size 1.27 1.27)) hide)
+    )

Commit message: Updated stuff that was needed to make Shipometer 23.04 case
Parts:
- C401, C405: Number on hand 24 -> 12
- U401: Number on hand 5 -> 4
Changed lines of the file:
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@@
       (effects (font (size 1.27 1.27)) hide)
     )
-    (property "Number on hand" "5" (at 129.54 96.52 0)
+    (property "Number on hand" "4" (at 129.54 96.52 0)
       (effects (font (size 1.27 1.27)) hide)
     )
@@
       (effects (font (size 1.27 1.27)) hide)
     )
-    (property "Number on hand" "24" (at 114.3 105.41 0)
+    (property "Number on hand" "12" (at 114.3 105.41 0)
       (effects (font (size 1.27 1.27)) hide)
     )
@@
       (effects (font (size 1.27 1.27)) hide)
     )
-    (property "Number on hand" "24" (at 144.78 109.22 0)
+    (property "Number on hand" "12" (at 144.78 109.22 0)
       (effects (font (size 1.27 1.27)) hide)
     )
