File: kicad/rollercoasterometer_hat_sf/rollercoasterometer_hat_sf.kicad_pcb (KiCad board)
At the start: 2 copper layers, 65 x 56.5 mm, 37 parts, among them J101 Raspberry_Pi_40, J102 Conn_01x03, J104 ICM20948, J105 BME280, J106 ZED-F9R, U102 74LS138, U1201 LPC2103, U401 TCR2EF 3.3V, U501 TCR2EF 1.8V, Y1201 12MHz

Commit message: As ordered on 03 Apr 2023. Some but not all numbers-on-hand have been updated.
Parts:
- removed R1, R144, R2: 68, Resistor_SMD:R_0603_1608Metric
- added R101: 68, KwanSystems:R_Array_Convex_4x0402, F.Cu at (205.5, 58.5)
- added R102: 68, KwanSystems:R_Array_Convex_4x0402, F.Cu at (205.5, 65.7)
Connections:
- D101 pad 1: /~{CS}_6D -> /~{CS}_6D+
- D103 pad 1: /~{CS}_PRES -> /~{CS}_PRES+
- D104 pad 1: /~{CS}_LPC_3V3 -> /~{CS}_LPC+
- D130 pad 1: /~{DRDY}_MAG_ECHO -> /DRDY_MAG-
- D141 pad 1: Net-(D141-K) -> /PPS-
- D144 pad 1: Net-(D144-K) -> /BOOTSTRAP-
- U102 pad 13: /~{CS}_LPC_3V3 -> /~{CS}_LPC
- U1201 pad 28: /~{CS}_LPC_3V3 -> /~{CS}_LPC
- U1201 pad 41: /Timer/PPS_ECHO -> /~{PPS}_ECHO
Routing:
- net /~{DRDY}_6D_ECHO: track 1.96 -> 71.2 mm, vias 0 -> 2
- net /DRDY-: track 67.2 -> 2.39 mm, vias 2 -> 0
- net /~{CS}_LPC_3V3: track 62.6 -> 0.00 mm, vias 5 -> 0
- net /~{CS}_LPC: track 0.00 -> 61.0 mm, vias 0 -> 5
- net /~{PPS}_ECHO: track 0.00 -> 53.0 mm, vias 0 -> 2
- net Net-(D141-K): track 49.2 -> 0.00 mm, vias 2 -> 0
- net Net-(D144-K): track 35.7 -> 0.00 mm, vias 2 -> 0
- net /LPC_~{BOOTSTRAP}: track 36.7 -> 72.2 mm, vias 3 -> 5
- net /~{CS}_PRES: track 38.9 -> 36.4 mm
- net /~{CS}_6D+: track 0.00 -> 2.39 mm
- net /PPS-: track 0.00 -> 2.39 mm
- net /Timer/PPS_ECHO: track 2.25 -> 0.00 mm
- net /BOOTSTRAP-: track 0.00 -> 1.52 mm
- net /~{CS}_LPC+: track 0.00 -> 1.52 mm
- net /~{CS}_PRES+: track 0.00 -> 1.52 mm
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