File: kicad/rollercoasterometer_hat_sf/rollercoasterometer_hat_timer.kicad_sch (KiCad schematic)
At the start: 7 parts, among them U1201 LPC2103, Y1201 12MHz

Commit message: Commit as-ordered shipometer 23.03
Parts:
- added D1206: Blue, LED_SMD:LED_0603_1608Metric, symbol Device:LED_Small
- added D1229: Red, LED_SMD:LED_0603_1608Metric, symbol Device:LED_Small
- added D1230: Green, LED_SMD:LED_0603_1608Metric, symbol Device:LED_Small
- added D1241, D1244: Yellow, LED_SMD:LED_0603_1608Metric, symbol Device:LED_Small
- added R1229, R1241, R1244: 68, Resistor_SMD:R_0402_1005Metric, symbol KwanSystems:RESISTOR
- C1205, C1217, C1240: Number on hand (none) -> 24
- C1211, C1212: Number on hand (none) -> 8
- U1201: Number on hand (none) -> 4
- Y1201: Number on hand (none) -> 1; Purpose (none) -> Timer crystal
Connections:
- net 1V8: no longer C1217.1, C1240.1, U1201.4 (VBAT)
- net DRDY: now also R1229.1
- net VDD(3V3): now also C1217.1, C1240.1, U1201.4 (VBAT), D1206.2 (A), D1241.2 (A), D1244.2 (A)
- net VSS: now also D1229.1 (K), D1230.1 (K)
- net ~{BOOTSTRAP}: now also R1244.1
- net ~{RESET}: now also D1206.1 (K)
- net DRDY_MAG_ECHO: now reaches U1201.30 ((RXD1/MAT2.2)P0.9)
- net DRDY_MAG_ECHO: now also D1230.2 (A)
- net PPS-: now reaches U1201.41 ((DTR1/MAT1.1)P0.13)
- net PPS-: now also R1241.1
- new net BOOSTSTRAP-: D1244.1 (K), R1244.2
- new net DRDY_6D_ECHO+: D1229.2 (A), R1229.2
- new net PPS+: D1241.1 (K), R1241.2
- no-connect marks 19 -> 20
Other:
- note added: "Bootstrap echo"
- note added: "DRDY_6D"
- note added: "DRDY_6D Echo"
- note added: "DRDY_MAG"
- note added: "DRDY_MAG echo"
- note added: "PPS"
- note added: "PPS Echo"
- note added: "Reset Echo"

Commit message: Updated to KiCad 7.0
Parts:
- D1206, D1230, D1241, D1244, R1229, R1241, R1244: Number in cart 10 -> (none); Number on hand 0 -> 10

Commit message: Added BME280 and ICM20948 stamps
Parts:
- removed D1206: Blue, LED_SMD:LED_0603_1608Metric, symbol Device:LED_Small
- removed D1229: Red, LED_SMD:LED_0603_1608Metric, symbol Device:LED_Small
- removed D1230: Green, LED_SMD:LED_0603_1608Metric, symbol Device:LED_Small
- removed D1241, D1244: Yellow, LED_SMD:LED_0603_1608Metric, symbol Device:LED_Small
- removed R1229, R1241, R1244: 68, Resistor_SMD:R_0402_1005Metric, symbol KwanSystems:RESISTOR
- C1205, C1211, C1212, C1217, C1240: footprint Capacitor_SMD:C_0402_1005Metric -> Capacitor_SMD:C_0603_1608Metric
Connections:
- net DRDY renamed ~{DRDY}_6D_ECHO
- net DRDY_MAG_ECHO renamed ~{DRDY}_MAG_ECHO
- net PPS- renamed PPS_ECHO
Other:
- note removed: "DRDY_6D Echo"
- note removed: "DRDY_MAG echo"
- note removed: "PPS Echo"
- note removed: "Reset Echo"
