File: kicad/shipomemter/shipometer.kicad_sch (KiCad schematic)
At the start: 25 parts, among them J101 Raspberry_Pi_40, J102 Conn_01x03, J104 ICM20948, J105 BME280, J106 ZED-F9R, U101 RaspberryPi 4B 2GB, U102 74LS138

Commit message: Updated numbers on hand and numbers in cart
Parts:
- C116: Number in cart (none) -> 24; Number on hand (none) -> 0
- D1230: Number on hand (none) -> 9
- J101: Mouser (none) -> 200-SSW12001TD; Number in cart (none) -> 1
- J106: Mouser (none) -> 571-1-215297-1; Number in cart (none) -> 2; Number on hand (none) -> 1
- R101, R102: Mouser (none) -> 667-EXB-28V680JX; Number in cart (none) -> 10; Number on hand (none) -> 0
Changed lines of the file:
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@@
+      (effects (font (size 1.27 1.27)) hide)
+    )
+    (property "Number in cart" "24" (at 45.72 142.24 0)
+      (effects (font (size 1.27 1.27)) hide)
+    )
+    (property "Number on hand" "0" (at 45.72 142.24 0)
       (effects (font (size 1.27 1.27)) hide)
     )
@@
     (property "Datasheet" "" (at 193.675 161.29 0)
       (effects (font (size 1.524 1.524)) hide)
+    )
+    (property "Mouser" "667-EXB-28V680JX" (at 182.88 153.67 0)
+      (effects (font (size 1.27 1.27)) hide)
+    )
+    (property "Number in cart" "10" (at 182.88 153.67 0)
+      (effects (font (size 1.27 1.27)) hide)
+    )
+    (property "Number on hand" "0" (at 182.88 153.67 0)
+      (effects (font (size 1.27 1.27)) hide)
     )
     (pin "1")
@@
       (effects (font (size 1.524 1.524)) hide)
     )
+    (property "Mouser" "667-EXB-28V680JX" (at 104.14 157.48 0)
+      (effects (font (size 1.27 1.27)) hide)
+    )
+    (property "Number in cart" "10" (at 104.14 157.48 0)
+      (effects (font (size 1.27 1.27)) hide)
+    )
+    (property "Number on hand" "0" (at 104.14 157.48 0)
+      (effects (font (size 1.27 1.27)) hide)
+    )
     (pin "1")
     (pin "8")
@@
       (effects (font (size 1.524 1.524)) hide)
     )
+    (property "Mouser" "667-EXB-28V680JX" (at 88.9 157.48 0)
+      (effects (font (size 1.27 1.27)) hide)
+    )
+    (property "Number in cart" "10" (at 88.9 157.48 0)
+      (effects (font (size 1.27 1.27)) hide)
+    )
+    (property "Number on hand" "0" (at 88.9 157.48 0)
+      (effects (font (size 1.27 1.27)) hide)
+    )
     (pin "1")
     (pin "8")
@@
     )
     (property "Datasheet" "" (at 219.71 115.57 0)
+      (effects (font (size 1.27 1.27)) hide)
+    )
+    (property "Number on hand" "1" (at 219.71 115.57 0)
+      (effects (font (size 1.27 1.27)) hide)
+    )
+    (property "Mouser" "571-1-215297-1" (at 219.71 115.57 0)
+      (effects (font (size 1.27 1.27)) hide)
+    )
+    (property "Number in cart" "2" (at 219.71 115.57 0)
       (effects (font (size 1.27 1.27)) hide)
     )
@@
       (effects (font (size 1.27 1.27)) hide)
     )
-    (property "Number in cart" "" (at 66.04 53.34 0)
+    (property "Number in cart" "1" (at 66.04 53.34 0)
       (effects (font (size 1.27 1.27)) hide)
     )
     (property "Number on hand" "0" (at 66.04 53.34 0)
+      (effects (font (size 1.27 1.27)) hide)
+    )
+    (property "Mouser" "200-SSW12001TD" (at 66.04 53.34 0)
       (effects (font (size 1.27 1.27)) hide)
     )
@@
       (effects (font (size 1.524 1.524)) hide)
     )
+    (property "Mouser" "667-EXB-28V680JX" (at 113.03 121.92 0)
+      (effects (font (size 1.27 1.27)) hide)
+    )
+    (property "Number in cart" "10" (at 113.03 121.92 0)
+      (effects (font (size 1.27 1.27)) hide)
+    )
+    (property "Number on hand" "0" (at 113.03 121.92 0)
+      (effects (font (size 1.27 1.27)) hide)
+    )
     (pin "1")
     (pin "8")
@@
       (effects (font (size 1.524 1.524)) hide)
     )
+    (property "Mouser" "667-EXB-28V680JX" (at 182.88 137.16 0)
+      (effects (font (size 1.27 1.27)) hide)
+    )
+    (property "Number in cart" "10" (at 182.88 137.16 0)
+      (effects (font (size 1.27 1.27)) hide)
+    )
+    (property "Number on hand" "0" (at 182.88 137.16 0)
+      (effects (font (size 1.27 1.27)) hide)
+    )
     (pin "1")
     (pin "8")
@@
       (effects (font (size 1.27 1.27)) hide)
     )
-    (property "Number on hand" "" (at 196.85 143.51 0)
+    (property "Number on hand" "9" (at 196.85 143.51 0)
       (effects (font (size 1.27 1.27)) hide)
     )
@@
     (property "Datasheet" "" (at 193.675 151.13 0)
       (effects (font (size 1.524 1.524)) hide)
+    )
+    (property "Mouser" "667-EXB-28V680JX" (at 182.88 143.51 0)
+      (effects (font (size 1.27 1.27)) hide)
+    )
+    (property "Number in cart" "10" (at 182.88 143.51 0)
+      (effects (font (size 1.27 1.27)) hide)
+    )
+    (property "Number on hand" "0" (at 182.88 143.51 0)
+      (effects (font (size 1.27 1.27)) hide)
     )
     (pin "1")
@@
       (effects (font (size 1.524 1.524)) hide)
     )
+    (property "Mouser" "667-EXB-28V680JX" (at 227.33 142.24 0)
+      (effects (font (size 1.27 1.27)) hide)
+    )
+    (property "Number in cart" "10" (at 227.33 142.24 0)
+      (effects (font (size 1.27 1.27)) hide)
+    )
+    (property "Number on hand" "0" (at 227.33 142.24 0)
+      (effects (font (size 1.27 1.27)) hide)
+    )
     (pin "1")
     (pin "8")
@@
       (effects (font (size 1.524 1.524)) hide)
     )
-    (pin "1")
+    (property "Mouser" "667-EXB-28V680JX" (at 99.06 157.48 0)
+      (effects (font (size 1.27 1.27)) hide)
+    )
+    (property "Number in cart" "10" (at 99.06 157.48 0)
+      (effects (font (size 1.27 1.27)) hide)
+    )
+    (property "Number on hand" "0" (at 99.06 157.48 0)
+      (effects (font (size 1.27 1.27)) hide)
+    )
+    (pin "1")

Commit message: Updated number on hand, and added more Digikey/Mouser/Mfg numbers
Parts:
- C116: Number in cart 24 -> (none); Number on hand 0 -> 24; Part Number (none) -> C0603C105K4PAC
- D101, D103, D104: Mouser (none) -> VLMW1300-GS08; Part Number (none) -> VLMW1300-GS08
- D1206: Mouser (none) -> 604-APT1608VBC/D; Part Number (none) -> APT1608VBC/D
- D1229: Mouser (none) -> 604-APT1608SURCK; Number on hand 2+2 -> 4; Part Number (none) -> APT1608SURCK
- D1230: Mouser (none) -> 604-APT1608ZGCK; Part Number (none) -> APT1608ZGCK
- D1241, D1244: Mouser (none) -> 604-APT1608SYCK; Part Number (none) -> APT1608SYCK
- J101: Number in cart 1 -> (none); Number on hand 0 -> 1; Part Number (none) -> SSW-120-01-G-D-LL
- J102: Part Number (none) -> PH1RB-03-UA
- J106: Digikey (none) -> A106613-ND; Number in cart 2 -> (none); Part Number (none) -> 1-215297-1
- R101, R102: Digikey (none) -> Y7680CT-ND; Number in cart 10 -> (none); Number on hand 0 -> 10; Part Number (none) -> EXB-28V680JX
- U101: Mouser (none) -> 358-SC01939
- U102: Digikey (none) -> 1727-4026-1-ND; Part Number (none) -> 74LVC138APW,118

Commit message: Updated stuff that was needed to make Shipometer 23.04 case
Parts:
- added R103: 10k, KwanSystems:R_Array_Convex_4x0402, symbol KwanSystems:RP4
- C116: Number on hand 24 -> 12
- D101, D103, D104: Number on hand 6 -> 3
- D1206, D1230: Number on hand 9 -> 8
- D1229: Number on hand 4 -> 3
- J101: footprint KwanSystems:PiHAT -> KwanSystems:PiHAT_NoSlot_Narrow; Digikey SSW-120-01-G-D-LL-ND -> 952-2150-ND; Number in cart (none) -> 1; Number on hand 1 -> 0; Part Number SSW-120-01-G-D-LL -> M20-7832046
- J102: Mouser (none) -> 649-68015-103HLF; Number in cart (none) -> 1; Number on hand 1 -> 0
- J106: Number in cart (none) -> 2; Number on hand 1 -> 0
- R101, R102: value 68 -> 330; Digikey Y7680CT-ND -> Y7331CT-ND; Mouser 667-EXB-28V680JX -> 667-EXB-28V331JX; Number in cart (none) -> 10; Number on hand 10 -> 0; Part Number EXB-28V680JX -> EXB-28V331JX
- U102: Number on hand 3 -> 2
Connections:
- net +3V3: now also R103.1 (4), R103.2 (4)
- net GND: now also R103.3 (4)
- net GPS_RX: now also J101.7 ((TX3)_GPIO4); no longer J101.29 (GPIO5)
- net GPS_TX: now also J101.29 ((RX3)_GPIO5); no longer J101.7 ((GCLK)_GPIO4)
- net GPS_~{RESET}: now also R103.8 (5)
- net LPC_~{BOOTSTRAP}: now also R103.6 (5)
- net LPC_~{RESET}: now also R102.1 (4), R103.7 (5); no longer D1206.1 (K)
- net LPC_RESET-: now reaches R102.8 (5)
- net LPC_RESET-: now also D1206.1 (K)
Other:
- removed sheet Stamp Tester
- moved on the sheet: R102A
