File: kicad/shipomemter/timer.kicad_sch (KiCad schematic)
At the start: 7 parts, among them U1201 LPC2103, Y1201 12MHz

Commit message: As ordered on 03 Apr 2023. Some but not all numbers-on-hand have been updated.
Parts:
- C605: renamed from C1205; value 100nF -> 1uF; Digikey 399-C0402C104K4RAC7411CT-ND -> 399-C0603C105K4PAC7411CT-ND; Mouser (none) -> 80-C0603C105K4PAC; Number on hand 24 -> (none)
- C611: renamed from C1211; Digikey 399-17554-1-ND -> 399-17583-1-ND; Number on hand 8 -> (none)
- C612: renamed from C1212; Digikey 399-17554-1-ND -> 399-17583-1-ND; Number on hand 8 -> (none)
- C617: renamed from C1217; value 100nF -> 1uF; Digikey 399-C0402C104K4RAC7411CT-ND -> 399-C0603C105K4PAC7411CT-ND; Mouser (none) -> 80-C0603C105K4PAC; Number on hand 24 -> (none)
- C640: renamed from C1240; value 100nF -> 1uF; Digikey 399-C0402C104K4RAC7411CT-ND -> 399-C0603C105K4PAC7411CT-ND; Mouser (none) -> 80-C0603C105K4PAC; Number on hand 24 -> (none)
- U601: renamed from U1201; Number on hand 4 -> (none)
- Y601: renamed from Y1201; Number on hand 1 -> 3

Commit message: Updated numbers on hand and numbers in cart
Parts:
- C605, C617, C640: Number in cart (none) -> 24; Number on hand (none) -> 0
- C611, C612: Mouser (none) -> 80-C0603C220F5G; Number in cart (none) -> 10; Number on hand (none) -> 0
- U601: Number on hand (none) -> 3
Changed lines of the file:
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@@
       (effects (font (size 1.27 1.27)) hide)
     )
-    (property "Number on hand" "" (at 49.53 152.4 0)
+    (property "Number on hand" "0" (at 49.53 152.4 0)
       (effects (font (size 1.27 1.27)) hide)
     )
@@
       (effects (font (size 1.27 1.27)) hide)
     )
+    (property "Number in cart" "24" (at 49.53 152.4 0)
+      (effects (font (size 1.27 1.27)) hide)
+    )
     (pin "1")
     (pin "2")
@@
       (effects (font (size 1.27 1.27)) hide)
     )
-    (property "Number on hand" "" (at 52.07 149.86 0)
+    (property "Number on hand" "0" (at 52.07 149.86 0)
       (effects (font (size 1.27 1.27)) hide)
     )
     (property "Mouser" "80-C0603C105K4PAC" (at 52.07 149.86 0)
+      (effects (font (size 1.27 1.27)) hide)
+    )
+    (property "Number in cart" "24" (at 52.07 149.86 0)
       (effects (font (size 1.27 1.27)) hide)
     )
@@
       (effects (font (size 1.27 1.27)) hide)
     )
-    (property "Number on hand" "" (at 52.07 96.52 0)
+    (property "Number on hand" "0" (at 52.07 96.52 0)
+      (effects (font (size 1.27 1.27)) hide)
+    )
+    (property "Number in cart" "10" (at 52.07 96.52 0)
+      (effects (font (size 1.27 1.27)) hide)
+    )
+    (property "Mouser" "80-C0603C220F5G" (at 52.07 96.52 0)
       (effects (font (size 1.27 1.27)) hide)
     )
@@
       (effects (font (size 1.27 1.27)) hide)
     )
-    (property "Number on hand" "" (at 52.07 88.9 0)
+    (property "Number on hand" "0" (at 52.07 88.9 0)
+      (effects (font (size 1.27 1.27)) hide)
+    )
+    (property "Number in cart" "10" (at 52.07 88.9 0)
+      (effects (font (size 1.27 1.27)) hide)
+    )
+    (property "Mouser" "80-C0603C220F5G" (at 52.07 88.9 0)
       (effects (font (size 1.27 1.27)) hide)
     )
@@
       (effects (font (size 1.27 1.27)) hide)
     )
-    (property "Number on hand" "" (at 69.85 104.14 0)
+    (property "Number on hand" "3" (at 69.85 104.14 0)
       (effects (font (size 1.27 1.27)) hide)
     )
@@
       (effects (font (size 1.27 1.27)) hide)
     )
-    (property "Number on hand" "" (at 54.61 152.4 0)
+    (property "Number on hand" "0" (at 54.61 152.4 0)
       (effects (font (size 1.27 1.27)) hide)
     )
@@
       (effects (font (size 1.27 1.27)) hide)
     )
+    (property "Number in cart" "24" (at 54.61 152.4 0)
+      (effects (font (size 1.27 1.27)) hide)
+    )

Commit message: Updated number on hand, and added more Digikey/Mouser/Mfg numbers
Parts:
- C605, C617, C640: Number in cart 24 -> (none); Number on hand 0 -> 24; Part Number (none) -> C0603C105K4PAC
- C611, C612: Number in cart 10 -> (none); Number on hand 0 -> 10; Part Number (none) -> C0603C220J5RAC
- U601: value LPC2103 -> LPC210x; Digikey 568-LPC2103FBD48EL-ND -> LPC2102FBD48,118-ND; Mouser (none) -> 771-LPC2102FBD48-S; Part Number (none) -> LPC2102FBD48,151
- Y601: Mouser (none) -> 815-ABM8G-12-18D2Y
Changed lines of the file:
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@@
       (effects (font (size 1.27 1.27)) hide)
     )
-    (property "Number on hand" "0" (at 49.53 152.4 0)
+    (property "Number on hand" "24" (at 49.53 152.4 0)
       (effects (font (size 1.27 1.27)) hide)
     )
@@
       (effects (font (size 1.27 1.27)) hide)
     )
-    (property "Number in cart" "24" (at 49.53 152.4 0)
+    (property "Number in cart" "" (at 49.53 152.4 0)
+      (effects (font (size 1.27 1.27)) hide)
+    )
+    (property "Part Number" "C0603C105K4PAC" (at 49.53 152.4 0)
       (effects (font (size 1.27 1.27)) hide)
     )
@@
       (effects (font (size 1.27 1.27)) hide)
     )
-    (property "Number on hand" "0" (at 52.07 149.86 0)
+    (property "Number on hand" "24" (at 52.07 149.86 0)
       (effects (font (size 1.27 1.27)) hide)
     )
@@
       (effects (font (size 1.27 1.27)) hide)
     )
-    (property "Number in cart" "24" (at 52.07 149.86 0)
+    (property "Number in cart" "" (at 52.07 149.86 0)
+      (effects (font (size 1.27 1.27)) hide)
+    )
+    (property "Part Number" "C0603C105K4PAC" (at 52.07 149.86 0)
       (effects (font (size 1.27 1.27)) hide)
     )
@@
     )
     (property "Purpose" "Timer crystal" (at 54.61 92.71 0)
+      (effects (font (size 1.27 1.27)) hide)
+    )
+    (property "Mouser" "815-ABM8G-12-18D2Y" (at 54.61 92.71 0)
       (effects (font (size 1.27 1.27)) hide)
     )
@@
       (effects (font (size 1.27 1.27)) hide)
     )
-    (property "Number on hand" "0" (at 52.07 96.52 0)
-      (effects (font (size 1.27 1.27)) hide)
-    )
-    (property "Number in cart" "10" (at 52.07 96.52 0)
+    (property "Number on hand" "10" (at 52.07 96.52 0)
+      (effects (font (size 1.27 1.27)) hide)
+    )
+    (property "Number in cart" "" (at 52.07 96.52 0)
       (effects (font (size 1.27 1.27)) hide)
     )
@@
       (effects (font (size 1.27 1.27)) hide)
     )
+    (property "Part Number" "C0603C220J5RAC" (at 52.07 96.52 0)
+      (effects (font (size 1.27 1.27)) hide)
+    )
     (pin "1")
     (pin "2")
@@
       (effects (font (size 1.27 1.27)) hide)
     )
-    (property "Number on hand" "0" (at 52.07 88.9 0)
-      (effects (font (size 1.27 1.27)) hide)
-    )
-    (property "Number in cart" "10" (at 52.07 88.9 0)
+    (property "Number on hand" "10" (at 52.07 88.9 0)
+      (effects (font (size 1.27 1.27)) hide)
+    )
+    (property "Number in cart" "" (at 52.07 88.9 0)
       (effects (font (size 1.27 1.27)) hide)
     )
     (property "Mouser" "80-C0603C220F5G" (at 52.07 88.9 0)
+      (effects (font (size 1.27 1.27)) hide)
+    )
+    (property "Part Number" "C0603C220J5RAC" (at 52.07 88.9 0)
       (effects (font (size 1.27 1.27)) hide)
     )
@@
       (effects (font (size 1.524 1.524)))
     )
-    (property "Value" "LPC2103" (at 102.87 68.58 0)
+    (property "Value" "LPC210x" (at 102.87 68.58 0)
       (effects (font (size 1.524 1.524)))
     )
@@
       (effects (font (size 1.524 1.524)) hide)
     )
-    (property "Digikey" "568-LPC2103FBD48EL-ND" (at 60.96 110.49 0)
+    (property "Digikey" "LPC2102FBD48,118-ND" (at 60.96 110.49 0)
       (effects (font (size 1.27 1.27)) hide)
     )
@@
     )
     (property "Number on hand" "3" (at 69.85 104.14 0)
+      (effects (font (size 1.27 1.27)) hide)
+    )
+    (property "Mouser" "771-LPC2102FBD48-S" (at 69.85 104.14 0)
+      (effects (font (size 1.27 1.27)) hide)
+    )
+    (property "Part Number" "LPC2102FBD48,151" (at 69.85 104.14 0)
       (effects (font (size 1.27 1.27)) hide)
     )
@@
       (effects (font (size 1.27 1.27)) hide)
     )
-    (property "Number on hand" "0" (at 54.61 152.4 0)
+    (property "Number on hand" "24" (at 54.61 152.4 0)
       (effects (font (size 1.27 1.27)) hide)
     )
@@
       (effects (font (size 1.27 1.27)) hide)
     )
-    (property "Number in cart" "24" (at 54.61 152.4 0)
-      (effects (font (size 1.27 1.27)) hide)
-    )
+    (property "Number in cart" "" (at 54.61 152.4 0)
+      (effects (font (size 1.27 1.27)) hide)
+    )
+    (property "Part Number" "C0603C105K4PAC" (at 54.61 152.4 0)
+      (effects (font (size 1.27 1.27)) hide)
+    )

Commit message: Updated stuff that was needed to make Shipometer 23.04 case
Parts:
- C605, C617, C640: Number on hand 24 -> 12
- C611, C612: Number on hand 10 -> 8
- U601, Y601: Number on hand 3 -> 2
Changed lines of the file:
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@@
       (effects (font (size 1.27 1.27)) hide)
     )
-    (property "Number on hand" "24" (at 49.53 152.4 0)
+    (property "Number on hand" "12" (at 49.53 152.4 0)
       (effects (font (size 1.27 1.27)) hide)
     )
@@
       (effects (font (size 1.27 1.27)) hide)
     )
-    (property "Number on hand" "24" (at 52.07 149.86 0)
+    (property "Number on hand" "12" (at 52.07 149.86 0)
       (effects (font (size 1.27 1.27)) hide)
     )
@@
       (effects (font (size 1.27 1.27)) hide)
     )
-    (property "Number on hand" "3" (at 54.61 92.71 0)
+    (property "Number on hand" "2" (at 54.61 92.71 0)
       (effects (font (size 1.27 1.27)) hide)
     )
@@
       (effects (font (size 1.27 1.27)) hide)
     )
-    (property "Number on hand" "10" (at 52.07 96.52 0)
+    (property "Number on hand" "8" (at 52.07 96.52 0)
       (effects (font (size 1.27 1.27)) hide)
     )
@@
       (effects (font (size 1.27 1.27)) hide)
     )
-    (property "Number on hand" "10" (at 52.07 88.9 0)
+    (property "Number on hand" "8" (at 52.07 88.9 0)
       (effects (font (size 1.27 1.27)) hide)
     )
@@
       (effects (font (size 1.27 1.27)) hide)
     )
-    (property "Number on hand" "3" (at 69.85 104.14 0)
+    (property "Number on hand" "2" (at 69.85 104.14 0)
       (effects (font (size 1.27 1.27)) hide)
     )
@@
       (effects (font (size 1.27 1.27)) hide)
     )
-    (property "Number on hand" "24" (at 54.61 152.4 0)
-      (effects (font (size 1.27 1.27)) hide)
-    )
+    (property "Number on hand" "12" (at 54.61 152.4 0)
+      (effects (font (size 1.27 1.27)) hide)
+    )
